File: docu/KiCad_sch/Instruction_decoder.kicad_sch (KiCad schematic)
At the start: 0 parts

Commit message: Update schema
Changed lines of the file:
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@@
 	(hierarchical_label "instruct_typ{0 - 2}"
 		(shape output)
-		(at 127 25.4 0)
+		(at 127 38.1 0)
 		(effects
 			(font
@@
 		)
 	)
-	(hierarchical_label "reg_use_f"
-		(shape output)
-		(at 127 76.2 0)
-		(effects
-			(font
-				(size 1.27 1.27)
-			)
-			(justify left)
-		)
-	)
 	(hierarchical_label "memory_use_f"
 		(shape output)
@@
 	(hierarchical_label "funct_3{0 - 2}"
 		(shape output)
-		(at 127 38.1 0)
+		(at 127 50.8 0)
 		(effects
 			(font
@@
 	(hierarchical_label "funct_7{0 - 6}"
 		(shape output)
-		(at 127 50.8 0)
+		(at 127 63.5 0)
 		(effects
 			(font
@@
 	(hierarchical_label "instruct{0 - 31}"
 		(shape input)
-		(at 76.2 25.4 180)
+		(at 76.2 38.1 180)
 		(effects
 			(font
@@
 	(hierarchical_label "jump_f"
 		(shape output)
-		(at 127 63.5 0)
+		(at 127 76.2 0)
 		(effects
 			(font
