File: docu/KiCad_sch/KiCad_sch.kicad_sch (KiCad schematic)
At the start: 0 parts

Commit message: Update schema
Other:
- sheet Instruction_decoder ports: added none; removed reg_use_f
Changed lines of the file:
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@@
-	(wire
-		(pts
-			(xy 313.69 121.92) (xy 313.69 172.72)
-		)
-		(stroke
-			(width 0)
-			(type default)
-		)
-	)
 	(wire
 		(pts
@@
 	(wire
 		(pts
-			(xy 313.69 121.92) (xy 382.27 121.92)
-		)
-		(stroke
-			(width 0)
-			(type default)
-		)
-	)
-	(wire
-		(pts
 			(xy 433.07 129.54) (xy 455.93 129.54)
 		)
@@
 		(pts
 			(xy 433.07 132.08) (xy 453.39 132.08)
-		)
-		(stroke
-			(width 0)
-			(type default)
-		)
-	)
-	(wire
-		(pts
-			(xy 313.69 172.72) (xy 293.37 172.72)
 		)
 		(stroke
@@
 			(effects
 				(font
-					(size 1.27 1.27)
-				)
-				(justify right)
-			)
-		)
-		(pin "reg_use_f" output
-			(at 293.37 172.72 0)
-			(effects
-				(font
